File: hardware/esp32s3-gnss-base-station.kicad_pcb (KiCad board)
At the start: 4 copper layers, 108 x 108 mm, 9 parts, among them SW1 SS-12D10L5

Commit message: Add KicCAD PCB Layout v0.1 and order on JLCPCB
Parts:
- removed mSDCard1: TF-001B, LCSC:TF-SMD_TF-001B
- added +3.3: TestPoint, TestPoint:TestPoint_Pad_D1.5mm, F.Cu at (94.8, 72.5)
- added B1: CR1220, LCSC:BAT-SMD_CR1220-2, F.Cu at (61.0, 85.8)
- added C1: 100nF, LCSC:C0402, F.Cu at (146.0, 93.5)
- added C10: 100nF, LCSC:C0402, F.Cu at (71.5, 91.8)
- added C11: 10uF, LCSC:C0603, F.Cu at (70.0, 91.6)
- added C12: 100nF, LCSC:C0402, F.Cu at (71.5, 98.3)
- added C13: 10uF, LCSC:C0603, F.Cu at (70.0, 98.5)
- added C14: 47pF, LCSC:C0603, F.Cu at (92.5, 91.8)
- added C2: 10uF, LCSC:C0603, F.Cu at (144.5, 93.7)
- added C3: 100nF, LCSC:C0402, F.Cu at (112.0, 129.6)
- added C4: 10uF, LCSC:C0603, F.Cu at (114.0, 129.7)
- added C5: 10uF, LCSC:C0603, F.Cu at (141.8, 82.2)
- added C6: 22uF, LCSC:C0805, F.Cu at (105.1, 72.5)
- added C7: 22uF, LCSC:C0805, F.Cu at (100.5, 72.5)
- added C8: 100nF, LCSC:C0402, F.Cu at (147.3, 115.5)
- added C9: 10uF, LCSC:C0603, F.Cu at (147.2, 117.0)
- added CN1: JST 2mm, LCSC:CONN-TH_B2B-PH-K-S, B.Cu at (138.0, 80.0)
- added J1: PWR_BYPASS, Connector_PinHeader_2.54mm:PinHeader_1x02_P2.54mm_Vertical, F.Cu at (119.5, 72.5)
- added J2: OLED, Connector_PinHeader_2.54mm:PinHeader_1x04_P2.54mm_Vertical, F.Cu at (77.6, 128.6)
- added L1: 2.2uH 2A 52mΩ, LCSC:IND-SMD_L4.0-W4.0, F.Cu at (96.4, 68.5)
- added L2: 120nH 110mA 2.66Ω, LCSC:L0402, F.Cu at (92.5, 99.5)
- added LED1: KT-0603R, LCSC:LED0603-RD, F.Cu at (117.5, 52.3)
- added LED2: KT-0603R, LCSC:LED0603-RD, F.Cu at (95.5, 52.3)
- added LED3: KT-0603R, LCSC:LED0603-RD, F.Cu at (83.5, 52.3)
- added LED4: KT-0603R, LCSC:LED0603-RD, F.Cu at (89.5, 52.3)
- added LED5: KT-0603R, LCSC:LED0603-RD, F.Cu at (116.2, 126.5)
- added Q1: MMDT3904, LCSC:SOT-363_L2.0-W1.3-P0.65-LS2.1-BR, F.Cu at (130.3, 85.3)
- added R1: 10k, LCSC:R0603, F.Cu at (142.0, 86.2)
- added R10: 10k, LCSC:R0603, F.Cu at (100.8, 65.5)
- added R11: 680k, LCSC:R0603, F.Cu at (107.2, 68.0)
- added R12: 150k, LCSC:R0603, F.Cu at (107.2, 65.5)
- added R13: 10k, LCSC:R0603, F.Cu at (132.0, 102.8)
- added R14: 10k, LCSC:R0603, F.Cu at (134.0, 103.8)
- added R15: 10k, LCSC:R0603, F.Cu at (136.0, 104.8)
- added R16: 10k, LCSC:R0603, F.Cu at (132.0, 108.8)
- added R17: 10k, LCSC:R0603, F.Cu at (134.0, 109.8)
- added R18: 10k, LCSC:R0603, F.Cu at (136.0, 110.8)
- added R19: 33, LCSC:R0603, F.Cu at (92.5, 95.2)
- added R2: 10k, LCSC:R0603, F.Cu at (128.0, 85.2)
- added R20: 1k, LCSC:R0603, F.Cu at (85.5, 56.8)
- added R21: 1k, LCSC:R0603, F.Cu at (87.5, 56.8)
- added R22: 1k, LCSC:R0603, F.Cu at (112.8, 126.5)
- added R3: 10k, LCSC:R0603, F.Cu at (130.2, 82.5)
- added R4: 10k, LCSC:R0603, F.Cu at (82.8, 107.4)
- added R5: 2.2k, LCSC:R0603, F.Cu at (148.5, 83.8)
- added R6: 2.2k, LCSC:R0603, F.Cu at (119.5, 56.8)
- added R7: 1k, LCSC:R0603, F.Cu at (98.8, 53.1)
- added R8: 150k, LCSC:R0603, F.Cu at (108.5, 108.8)
- added R9: 150k, LCSC:R0603, F.Cu at (107.0, 108.8)
- added SDCard1: TF-001B, LCSC:TF-SMD_TF-001B, F.Cu at (146.0, 106.5)
- added U1: ESP32-S3-WROOM-1-N16R8, LCSC:ESP32-S3-WROOM-1, F.Cu at (100.0, 125.0)
- added U2: ZED-F9P-04B, RF_GPS:ublox_ZED, F.Cu at (82.5, 94.0)
- added U3: CP2102-GMR, LCSC:WQFN-28_L5.0-W5.0-P0.50-BL-EP3.2, F.Cu at (138.0, 86.0)
- added U4: TP4054, LCSC:SOT-23-5_L3.0-W1.7-P0.95-LS2.8-BL, F.Cu at (145.4, 83.3)
- added U5: SY8089AAAC, LCSC:SOT-23-5_L3.0-W1.7-P0.95-LS2.8-BR, F.Cu at (102.8, 69.0)
- added U6: BWMCX-KE, LCSC:SMA-TH_BWMCX-KE, F.Cu at (100.0, 100.0)
Connections:
- SW1 pad 1: unconnected-(SW1-Pad1) -> Net-(U4-BAT)
- SW1 pad 2: unconnected-(SW1-Pad2) -> +BATT
- USB1 pad 1: unconnected-(USB1-VBUS-Pad1) -> +5V
- USB1 pad 2: unconnected-(USB1-D--Pad2) -> Net-(U3-D-)
- USB1 pad 3: unconnected-(USB1-D+-Pad3) -> Net-(U3-D+)
- USB1 pad 5: unconnected-(USB1-GND-Pad5) -> GND
- USB1 pad 6: unconnected-(USB1-SH1-Pad6) -> GND
- USB1 pad 7: unconnected-(USB1-SH2-Pad7) -> GND
- USB1 pad 8: unconnected-(USB1-SH3-Pad8) -> GND
- USB1 pad 9: unconnected-(USB1-SH4-Pad9) -> GND
Routing:
- net +3V3: track 0.00 -> 300.0 mm, vias 0 -> 15
- net ENABLE: track 0.00 -> 101.1 mm, vias 0 -> 3
- net +BATT: track 0.00 -> 81.5 mm, vias 0 -> 1
- net +5V: track 0.00 -> 74.0 mm, vias 0 -> 2
- net COM_RX: track 0.00 -> 72.2 mm, vias 0 -> 2
- net COM_TX: track 0.00 -> 71.1 mm, vias 0 -> 2
- net BOOT: track 0.00 -> 58.4 mm, vias 0 -> 3
- net Net-(U2-TIMEPULSE): track 0.00 -> 51.1 mm, vias 0 -> 2
- net SD_CMD: track 0.00 -> 49.7 mm
- net Net-(U4-BAT): track 0.00 -> 49.6 mm
- net SD_IO3: track 0.00 -> 49.2 mm
- net SD_IO1: track 0.00 -> 48.6 mm
- net SD_IO2: track 0.00 -> 48.5 mm
- net SD_IO0: track 0.00 -> 48.4 mm
- net SD_CLK: track 0.00 -> 46.9 mm
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- added copper zone on B.Cu, net GND
- added copper zone on F.Cu, net GND
- added copper zone on In1.Cu, net GND
- added copper zone on In2.Cu, net GND
Other:
- board text added: "+"
- board text added: "3V3"
- board text added: "BAT+"
- board text added: "GND"
- board text added: "GNSS Base Station V1.1"
- board text added: "SCL"
- board text added: "SDA"
- board text added: "TP+4.2"
- board text added: "TP+5.0"
- board text added: "["
- board text added: "]"

Commit message: Update PCB and export some images
Changed lines of the file:
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@@
 			(crossoutdnponfab yes)
 			(subtractmaskfromsilk no)
-			(outputformat 1)
+			(outputformat 5)
 			(mirror no)
-			(drillshape 1)
+			(drillshape 0)
 			(scaleselection 1)
 			(outputdirectory "")
@@
 		)
 		(embedded_fonts no)
-		(model "${KICAD9_3DMODEL_DIR}/RF_GPS.3dshapes/ublox_ZED.step"
+		(model "${KIPRJMOD}/libs/LCSC.3dshapes/LCC-LGA-102_L22.0-W17.0_FM660.wrl"
 			(offset
 				(xyz 0 0 0)
@@
 			)
 			(rotate
-				(xyz 0 0 0)
+				(xyz -0 -0 90)
 			)
 		)
@@
 	)
 	(footprint "LCSC:TF-SMD_TF-001B"
+		(locked yes)
 		(layer "F.Cu")
 		(at 146 106.5 180)
@@
 		(polygon
 			(pts
-				(xy 40 40) (xy 160 40) (xy 160 131.8) (xy 40 131.8)
+				(xy 40 45) (xy 160 45) (xy 160 131.8) (xy 40 131.8)
 			)
 		)
